Commit message: moving success but only gripper1

File: HYU_ur5e_robotiq/src/robotiq_85_gripper/robotiq_85_description/urdf/robotiq_85_gripper.transmission.xacro (robot description, xacro)
@@ -5,9 +5,9 @@
             <type>transmission_interface/SimpleTransmission</type>
             <joint name="${prefix}gripper_finger1_joint">
-                <hardwareInterface>PositionJointInterface</hardwareInterface>
+                <hardwareInterface>hardware_interface/EffortJointInterface</hardwareInterface>
             </joint>
             <actuator name="${prefix}gripper_finger1_motor">
                 <mechanicalReduction>1</mechanicalReduction>
-                <hardwareInterface>PositionJointInterface</hardwareInterface>
+                <hardwareInterface>hardware_interface/EffortJointInterface</hardwareInterface>
             </actuator>
         </transmission>

File: universal_robot/ur_description/urdf/inc/ur5e_macro.xacro (robot description, xacro)
@@ -23,5 +23,5 @@
    physical_parameters_file:='$(find ur_description)/config/ur5e/physical_parameters.yaml'
    visual_parameters_file:='$(find ur_description)/config/ur5e/visual_parameters.yaml'
-   transmission_hw_interface:=hardware_interface/PositionJointInterface
+   transmission_hw_interface:=hardware_interface/EffortJointInterface
    safety_limits:=false
    safety_pos_margin:=0.15

File: ur5e_robotiq_description/urdf/ur5e_gripper.xacro (robot description, xacro)
@@ -1,17 +1,4 @@
 <?xml version="1.0"?>
 <robot xmlns:xacro="http://wiki.ros.org/xacro" name="ur5e_robot">
-  <!--
-    This is a convenience top-level xacro which loads the macro for the UR5e
-    which defines the default values for the various "parameters files"
-    parameters for a UR5e.
-    This file is only useful when loading a stand-alone, completely isolated
-    robot with only default values for all parameters such as the kinematics,
-    visual and physical parameters and joint limits.
-    This file is not intended to be integrated into a larger scene or other
-    composite xacro.
-    Instead, xacro:include 'inc/ur5e_macro.xacro' and override the defaults
-    for the arguments to that macro.
-    Refer to 'inc/ur_macro.xacro' for more information.
-  -->
     <xacro:property name="PI" value="3.1415926535897931"/>
   <xacro:include filename="$(find ur_description)/urdf/inc/ur5e_macro.xacro"/>
@@ -21,5 +8,5 @@
   <!-- gripper -->
   <xacro:robotiq_85_gripper prefix="" parent="tool0">
-    <origin xyz="0 0 0" rpy="0 0 -${PI/2}"/>
+    <origin xyz="0 0 0" rpy="0 0 0"/>
   </xacro:robotiq_85_gripper>
 </robot>
