Commit message: change to ur5e_robotiq_moveit_config

File: ur5e_robotiq_moveit_config/config/gazebo_ur5e_robot.urdf (robot description, URDF)
Before this commit: robot ur5e_robot, 21 links, 20 joints
Joints:
- joint gripper_finger1_joint: limit lower=0.0 upper=0.804 effort=1000 velocity=2.0 -> lower=-0.8757 upper=0.8757 effort=1000 velocity=2.0
